File: CleverCoffee_ESP32/CleverCoffee_ESP32.kicad_pcb (KiCad board)
At the start: 2 copper layers, 95 x 65 mm, 32 parts

Commit message: Bugfix Lable Silkscreen
E_TRIG change VCC to 5V
P_SW change GND to 3,3V
W_SENS change IO36 to IO23
P_SENS change IO23 to IO36
ROTRAY SWITCH CLK DT
change all VCC to 3,3V

Change REV to 1.4
Other:
- board text added: "3,3V"
- board text added: "CleverCoffee ESP32 Rev 1.4"
- board text removed: "CleverCoffee ESP32 Rev 1.3"
- board text removed: "VCC"
Changed lines of the file:
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@@
       (connect_pads (clearance 0))
       (min_thickness 0.254)
-      (keepout (tracks not_allowed) (vias not_allowed) (pads not_allowed ) (copperpour allowed) (footprints allowed))
+      (keepout (tracks not_allowed) (vias not_allowed) (pads not_allowed) (copperpour allowed) (footprints allowed))
       (fill (thermal_gap 0.508) (thermal_bridge_width 0.508))
       (polygon
@@
     (effects (font (size 0.5 0.5) (thickness 0.1)))
   )
-  (gr_text "VCC" (at 187.38 118.4 90) (layer "F.SilkS")
+  (gr_text "3,3V" (at 187.38 118.4 90) (layer "F.SilkS")
     (effects (font (size 0.5 0.5) (thickness 0.1)))
   )
@@
     (effects (font (size 0.5 0.5) (thickness 0.1)))
   )
-  (gr_text "CleverCoffee ESP32 Rev 1.3" (at 158.13 101.04) (layer "F.SilkS")
+  (gr_text "CleverCoffee ESP32 Rev 1.4\n" (at 158.13 101.04) (layer "F.SilkS")
     (effects (font (size 1 1) (thickness 0.15)))
   )
@@
     (effects (font (size 0.5 0.5) (thickness 0.1)))
   )
-  (gr_text "DT" (at 187.39 111.64 90) (layer "F.SilkS")
-    (effects (font (size 0.5 0.5) (thickness 0.1)))
-  )
-  (gr_text "GND" (at 187.38 127.46 90) (layer "F.SilkS")
+  (gr_text "CLK" (at 187.39 111.64 90) (layer "F.SilkS")
+    (effects (font (size 0.5 0.5) (thickness 0.1)))
+  )
+  (gr_text "3,3V\n" (at 187.38 127.46 90) (layer "F.SilkS")
     (effects (font (size 0.5 0.5) (thickness 0.1)))
   )
@@
     (effects (font (size 0.5 0.5) (thickness 0.1)))
   )
-  (gr_text "CLK" (at 187.38 109.12 90) (layer "F.SilkS")
+  (gr_text "DT" (at 187.38 109.12 90) (layer "F.SilkS")
     (effects (font (size 0.5 0.5) (thickness 0.1)))
   )
@@
     (effects (font (size 0.5 0.5) (thickness 0.1)))
   )
-  (gr_text "VCC" (at 107.3 102.56 270) (layer "F.SilkS")
-    (effects (font (size 0.5 0.5) (thickness 0.1)))
-  )
-  (gr_text "VCC" (at 117.83 132.435) (layer "F.SilkS")
+  (gr_text "5V\n" (at 107.3 102.56 270) (layer "F.SilkS")
+    (effects (font (size 0.5 0.5) (thickness 0.1)))
+  )
+  (gr_text "3,3V" (at 117.83 132.435) (layer "F.SilkS")
     (effects (font (size 0.5 0.5) (thickness 0.1)))
   )
@@
     (effects (font (size 0.5 0.5) (thickness 0.1)))
   )
-  (gr_text "IO36\n\n" (at 133.69 132.845) (layer "F.SilkS")
+  (gr_text "IO23\n\n" (at 133.69 132.845) (layer "F.SilkS")
     (effects (font (size 0.5 0.5) (thickness 0.1)))
   )
@@
     (effects (font (size 0.5 0.5) (thickness 0.1)))
   )
-  (gr_text "IO23\n" (at 151.95 132.435) (layer "F.SilkS")
-    (effects (font (size 0.5 0.5) (thickness 0.1)))
-  )
+  (gr_text "IO36\n" (at 151.95 132.435) (layer "F.SilkS")
+    (effects (font (size 0.5 0.5) (thickness 0.1)))
+  )
